File: hardware/base/Untitled.brd (EAGLE design)
At the start: 83.2 x 83.2 mm, 29 parts, among them Q1 IRLML2502, Q2 IRLML2502, Q3 IRLML2502, Q4 IRLML2502, U2 MIC5205

Commit message: update
Parts:
- moved FTDI 1.27 mm to (39.4, 27.9)
- moved U$3 1.27 mm to (39.4, 39.4)
Changed lines of the file:
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@@
 <attribute name="VALUE" x="44.958" y="32.5755" size="0.4064" layer="27" rot="R90"/>
 </element>
-<element name="FTDI" library="SparkFun-Connectors" package="FTDI_DEVICE_SIDE" value="FTDI_DEVICE" x="40.64" y="27.94" smashed="yes" rot="R180">
-<attribute name="VALUE" x="52.07" y="31.115" size="1.27" layer="27" rot="R180"/>
+<element name="FTDI" library="SparkFun-Connectors" package="FTDI_DEVICE_SIDE" value="FTDI_DEVICE" x="39.37" y="27.94" smashed="yes" rot="R180">
+<attribute name="VALUE" x="50.8" y="31.115" size="1.27" layer="27" rot="R180"/>
 </element>
 <element name="POWER" library="SparkFun-Connectors" package="1X02" value="" x="25.4" y="53.34" smashed="yes" rot="R45">
@@
 <element name="C2" library="SparkFun-Capacitors" package="0402-CAP" value="0.1uF" x="37.465" y="52.705" rot="R180"/>
 <element name="R1" library="SparkFun-Passives" package="0402-RES" value="1K" x="29.21" y="31.75" rot="R90"/>
-<element name="U$3" library="esp8266modules" package="ESP12" value="ESP12" x="40.64" y="39.37" rot="MR0"/>
+<element name="U$3" library="esp8266modules" package="ESP12" value="ESP12" x="39.37" y="39.37" rot="MR0"/>
 </elements>
 <signals>
@@
 <wire x1="36.815" y1="52.705" x2="37.3038" y2="40.6267" width="0" layer="19" extent="1-1"/>
 <wire x1="33.02" y1="49.4" x2="36.815" y2="52.705" width="0" layer="19" extent="1-1"/>
-<wire x1="34.29" y1="27.94" x2="33.02" y2="49.4" width="0" layer="19" extent="1-1"/>
-<wire x1="36.83" y1="27.94" x2="34.29" y2="27.94" width="0" layer="19" extent="1-1"/>
+<wire x1="33.02" y1="27.94" x2="33.02" y2="49.4" width="0" layer="19" extent="1-1"/>
+<wire x1="35.56" y1="27.94" x2="33.02" y2="27.94" width="0" layer="19" extent="1-1"/>
 <wire x1="41.275" y1="32.37" x2="40.1496" y2="37.2484" width="0" layer="19" extent="1-1"/>
 <wire x1="43.815" y1="32.37" x2="41.275" y2="32.37" width="0" layer="19" extent="1-1"/>
 <wire x1="46.355" y1="32.37" x2="43.815" y2="32.37" width="0" layer="19" extent="1-1"/>
 <wire x1="25.4" y1="53.34" x2="33.02" y2="49.4" width="0" layer="19" extent="1-1"/>
-<wire x1="18.590378125" y1="63.95961875" x2="34.29" y2="27.94" width="0" layer="19" extent="1-1"/>
+<wire x1="18.590378125" y1="63.95961875" x2="33.02" y2="27.94" width="0" layer="19" extent="1-1"/>
 <wire x1="15.41956875" y1="65.93393125" x2="18.590378125" y2="63.95961875" width="0" layer="19" extent="1-1"/>
 <wire x1="16.050378125" y1="18.590378125" x2="25.4" y2="53.34" width="0" layer="19" extent="1-1"/>
 <wire x1="14.076065625" y1="15.41956875" x2="16.050378125" y2="18.590378125" width="0" layer="19" extent="1-1"/>
 <wire x1="29.21" y1="31.1" x2="14.076065625" y2="15.41956875" width="0" layer="19" extent="1-1"/>
-<wire x1="33.74" y1="31.17" x2="29.21" y2="31.1" width="0" layer="19" extent="1-1"/>
+<wire x1="32.47" y1="31.17" x2="29.21" y2="31.1" width="0" layer="19" extent="1-1"/>
 <wire x1="61.41961875" y1="16.050378125" x2="46.355" y2="32.37" width="0" layer="19" extent="1-1"/>
 <wire x1="64.590428125" y1="14.076065625" x2="61.41961875" y2="16.050378125" width="0" layer="19" extent="1-1"/>
@@
 <contactref element="FTDI" pad="P$1"/>
 <contactref element="U$3" pad="GPIO0"/>
-<wire x1="33.74" y1="37.17" x2="46.99" y2="27.94" width="0" layer="19" extent="1-1"/>
+<wire x1="32.47" y1="37.17" x2="45.72" y2="27.94" width="0" layer="19" extent="1-1"/>
 </signal>
 <signal name="SCL">
@@
 <contactref element="U$3" pad="GPIO4"/>
 <wire x1="38.735" y1="32.37" x2="38.6079" y2="41.4516" width="0" layer="19" extent="1-1"/>
-<wire x1="33.74" y1="41.17" x2="38.735" y2="32.37" width="0" layer="19" extent="1-1"/>
+<wire x1="32.47" y1="41.17" x2="38.735" y2="32.37" width="0" layer="19" extent="1-1"/>
 </signal>
 <signal name="N$32">
@@
 <wire x1="38.7651" y1="50.48" x2="70.485" y2="68.58" width="0" layer="19" extent="1-1"/>
 <wire x1="38.7651" y1="48.58" x2="38.7651" y2="50.48" width="0" layer="19" extent="1-1"/>
-<wire x1="39.37" y1="27.94" x2="38.7651" y2="48.58" width="0" layer="19" extent="1-1"/>
+<wire x1="38.1" y1="27.94" x2="38.7651" y2="48.58" width="0" layer="19" extent="1-1"/>
 <wire x1="27.19605" y1="55.13605" x2="38.7651" y2="48.58" width="0" layer="19" extent="1-1"/>
 <wire x1="9.525" y1="68.58" x2="27.19605" y2="55.13605" width="0" layer="19" extent="1-1"/>
 <wire x1="9.525" y1="11.43" x2="27.19605" y2="55.13605" width="0" layer="19" extent="1-1"/>
-<wire x1="47.74" y1="43.17" x2="9.525" y2="11.43" width="0" layer="19" extent="1-1"/>
+<wire x1="46.47" y1="43.17" x2="9.525" y2="11.43" width="0" layer="19" extent="1-1"/>
 <wire x1="70.485" y1="11.43" x2="38.7651" y2="50.48" width="0" layer="19" extent="1-1"/>
 </signal>
@@
 <contactref element="U$3" pad="GPIO5"/>
 <wire x1="36.195" y1="33.67" x2="38.1033" y2="41.4516" width="0" layer="19" extent="1-1"/>
-<wire x1="33.74" y1="39.17" x2="36.195" y2="33.67" width="0" layer="19" extent="1-1"/>
+<wire x1="32.47" y1="39.17" x2="36.195" y2="33.67" width="0" layer="19" extent="1-1"/>
 </signal>
 <signal name="N$38">
@@
 <contactref element="U$3" pad="GPIO16"/>
 <wire x1="63.040378125" y1="60.500378125" x2="60.500378125" y2="63.040378125" width="0" layer="19" extent="1-1"/>
-<wire x1="47.74" y1="39.17" x2="60.500378125" y2="63.040378125" width="0" layer="19" extent="1-1"/>
+<wire x1="46.47" y1="39.17" x2="60.500378125" y2="63.040378125" width="0" layer="19" extent="1-1"/>
 </signal>
 <signal name="M3">
@@
 <contactref element="U$3" pad="GPIO13"/>
 <wire x1="60.500378125" y1="16.96961875" x2="63.95961875" y2="18.590378125" width="0" layer="19" extent="1-1"/>
-<wire x1="47.74" y1="33.17" x2="60.500378125" y2="16.96961875" width="0" layer="19" extent="1-1"/>
+<wire x1="46.47" y1="33.17" x2="60.500378125" y2="16.96961875" width="0" layer="19" extent="1-1"/>
 </signal>
 <signal name="M2">
@@
 <contactref element="U$3" pad="GPIO12"/>
 <wire x1="16.96961875" y1="19.50961875" x2="18.590378125" y2="16.050378125" width="0" layer="19" extent="1-1"/>
-<wire x1="47.74" y1="35.17" x2="16.96961875" y2="19.50961875" width="0" layer="19" extent="1-1"/>
+<wire x1="46.47" y1="35.17" x2="16.96961875" y2="19.50961875" width="0" layer="19" extent="1-1"/>
 </signal>
 <signal name="M1">
@@
 <contactref element="U$3" pad="GPIO14"/>
 <wire x1="16.050378125" y1="61.41961875" x2="19.50961875" y2="63.040378125" width="0" layer="19" extent="1-1"/>
-<wire x1="47.74" y1="37.17" x2="16.050378125" y2="61.41961875" width="0" layer="19" extent="1-1"/>
+<wire x1="46.47" y1="37.17" x2="16.050378125" y2="61.41961875" width="0" layer="19" extent="1-1"/>
 </signal>
 <signal name="N$3">
@@
 <wire x1="38.735" y1="33.67" x2="41.4562" y2="38.0733" width="0" layer="19" extent="1-1"/>
 <wire x1="36.195" y1="32.37" x2="38.735" y2="33.67" width="0" layer="19" extent="1-1"/>
-<wire x1="33.74" y1="35.17" x2="36.195" y2="32.37" width="0" layer="19" extent="1-1"/>
-<wire x1="47.74" y1="31.17" x2="33.74" y2="35.17" width="0" layer="19" extent="1-1"/>
-<wire x1="47.74" y1="41.17" x2="47.74" y2="31.17" width="0" layer="19" extent="1-1"/>
+<wire x1="32.47" y1="35.17" x2="36.195" y2="32.37" width="0" layer="19" extent="1-1"/>
+<wire x1="46.47" y1="31.17" x2="32.47" y2="35.17" width="0" layer="19" extent="1-1"/>
+<wire x1="46.47" y1="41.17" x2="46.47" y2="31.17" width="0" layer="19" extent="1-1"/>
 </signal>
 <signal name="N$1">
@@
 <contactref element="FTDI" pad="P$2"/>
 <contactref element="U$3" pad="RX"/>
-<wire x1="33.74" y1="43.17" x2="44.45" y2="27.94" width="0" layer="19" extent="1-1"/>
+<wire x1="32.47" y1="43.17" x2="43.18" y2="27.94" width="0" layer="19" extent="1-1"/>
 </signal>
 <signal name="TX">
 <contactref element="FTDI" pad="P$3"/>
 <contactref element="U$3" pad="TX"/>
-<wire x1="33.74" y1="45.17" x2="41.91" y2="27.94" width="0" layer="19" extent="1-1"/>
+<wire x1="32.47" y1="45.17" x2="40.64" y2="27.94" width="0" layer="19" extent="1-1"/>
 </signal>
 <signal name="N$20">
 <contactref element="U$3" pad="GPIO15"/>
 <contactref element="R1" pad="2"/>
-<wire x1="29.21" y1="32.4" x2="33.74" y2="33.17" width="0" layer="19" extent="1-1"/>
+<wire x1="29.21" y1="32.4" x2="32.47" y2="33.17" width="0" layer="19" extent="1-1"/>
 </signal>
 </signals>
