File: hardware/Flying5 v1.0 - schematic design/Untitled.brd (EAGLE design)
At the start: 83.2 x 83.2 mm, 30 parts, among them Q1 IRLML2502, Q2 IRLML2502, Q3 IRLML2502, Q4 IRLML2502, U2 MIC5205

Commit message: pcb update
Parts:
- moved C10 2.54 mm to (43.8, 33.0)
- moved C6 2.54 mm to (41.3, 33.0)
- moved U2 1.27 mm to (30.5, 47.6)
- moved R1 1.27 mm to (29.2, 30.5), turned to 180 degrees
- turned C2 to 180 degrees
- turned R12 to 135 degrees
- turned R4 to 90 degrees
- turned R9 to 225 degrees
Routing:
- net GND: track 27.2 -> 130.2 mm
- net M4: track 0.00 -> 33.0 mm
- net 3.3V: track 0.00 -> 20.4 mm
- net SDA: track 0.00 -> 13.3 mm
- net N$5: track 0.00 -> 9.61 mm, vias 0 -> 2
- net SCL: track 0.00 -> 8.40 mm
- net N$20: track 0.00 -> 7.40 mm
- net VCC: track 194.3 -> 201.1 mm, vias 1 -> 3
- net N$29: track 0.00 -> 3.73 mm
- net N$40: track 0.00 -> 3.66 mm
- net N$39: track 0.00 -> 3.66 mm
- net N$38: track 0.00 -> 3.40 mm
- net M2: track 0.00 -> 1.80 mm
- net M3: track 0.00 -> 1.80 mm
- net M1: track 0.00 -> 1.80 mm

Commit message: pcb update
Routing:
- net GND: track 130.2 -> 174.2 mm
- net DTR: track 0.00 -> 22.5 mm, vias 0 -> 2
- net 3.3V: track 20.4 -> 37.7 mm
- net N$32: track 0.00 -> 12.2 mm, vias 0 -> 2
- net VCC: track 201.1 -> 207.1 mm
- net SCL: track 8.40 -> 9.96 mm, vias 0 -> 1
- net M4: track 33.0 -> 31.9 mm
Changed lines of the file:
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@@
 <wire x1="62.05461875" y1="16.685378125" x2="62.05461875" y2="16.33461875" width="1.016" layer="1"/>
 <wire x1="62.05461875" y1="16.33461875" x2="60.96" y2="15.24" width="1.016" layer="1"/>
-<wire x1="60.96" y1="15.24" x2="50.165" y2="26.035" width="1.016" layer="1"/>
+<wire x1="60.96" y1="15.24" x2="53.34" y2="22.86" width="1.016" layer="1"/>
+<wire x1="53.34" y1="22.86" x2="50.165" y2="26.035" width="1.016" layer="1"/>
 <wire x1="50.165" y1="26.035" x2="37.465" y2="26.035" width="1.016" layer="1"/>
 <wire x1="37.465" y1="26.035" x2="36.83" y2="26.67" width="1.016" layer="1"/>
@@
 <wire x1="29.845" y1="47.625" x2="30.48" y2="48.26" width="0.6096" layer="1"/>
 <wire x1="30.48" y1="48.26" x2="30.48" y2="48.9251" width="0.6096" layer="1"/>
-<wire x1="42.7262" y1="40.6267" x2="63.32461875" y2="62.05461875" width="0" layer="19" extent="1-1"/>
+<wire x1="63.32461875" y1="62.05461875" x2="64.135" y2="61.2442375" width="0.4064" layer="1"/>
+<wire x1="64.135" y1="61.2442375" x2="64.135" y2="60.96" width="0.4064" layer="1"/>
+<wire x1="64.135" y1="60.96" x2="53.34" y2="50.165" width="0.4064" layer="1"/>
+<wire x1="53.34" y1="50.165" x2="53.34" y2="22.86" width="0.4064" layer="1"/>
 <wire x1="41.4196" y1="37.2484" x2="42.7262" y2="40.6267" width="0" layer="19" extent="1-1"/>
 <wire x1="38.5738" y1="40.6267" x2="42.7262" y2="40.6267" width="0" layer="19" extent="1-1"/>
@@
 <contactref element="FTDI" pad="P$1"/>
 <contactref element="U$3" pad="GPIO0"/>
-<wire x1="33.74" y1="37.17" x2="46.99" y2="27.94" width="0" layer="19" extent="1-1"/>
+<wire x1="33.74" y1="37.17" x2="35.56" y2="35.35" width="0.4064" layer="16"/>
+<wire x1="35.56" y1="35.35" x2="35.56" y2="30.48" width="0.4064" layer="16"/>
+<via x="35.56" y="30.48" extent="1-16" drill="0.6"/>
+<wire x1="35.56" y1="30.48" x2="36.195" y2="31.115" width="0.4064" layer="1"/>
+<wire x1="36.195" y1="31.115" x2="39.37" y2="31.115" width="0.4064" layer="1"/>
+<wire x1="39.37" y1="31.115" x2="40.005" y2="31.75" width="0.4064" layer="1"/>
+<via x="40.005" y="31.75" extent="1-16" drill="0.6"/>
+<wire x1="40.005" y1="31.75" x2="41.275" y2="30.48" width="0.4064" layer="16"/>
+<wire x1="41.275" y1="30.48" x2="46.99" y2="30.48" width="0.4064" layer="16"/>
+<wire x1="46.99" y1="30.48" x2="46.99" y2="27.94" width="0.4064" layer="16"/>
 </signal>
 <signal name="SCL">
@@
 <contactref element="R4" pad="2"/>
 <contactref element="U$3" pad="GPIO4"/>
-<wire x1="33.74" y1="41.17" x2="36.09" y2="41.17" width="0.4064" layer="1"/>
-<wire x1="36.09" y1="41.17" x2="38.1" y2="43.18" width="0.4064" layer="1"/>
-<wire x1="38.1" y1="43.18" x2="39.37" y2="43.18" width="0.4064" layer="1"/>
-<wire x1="39.37" y1="43.18" x2="39.8779" y2="42.6721" width="0.4064" layer="1"/>
-<wire x1="39.8779" y1="42.6721" x2="39.8779" y2="41.4516" width="0.4064" layer="1"/>
-<wire x1="38.735" y1="33.67" x2="39.8779" y2="41.4516" width="0" layer="19" extent="1-1"/>
+<wire x1="38.735" y1="33.67" x2="36.21" y2="36.195" width="0.4064" layer="1"/>
+<wire x1="36.21" y1="36.195" x2="36.195" y2="36.195" width="0.4064" layer="1"/>
+<via x="36.195" y="36.195" extent="1-16" drill="0.6"/>
+<wire x1="36.195" y1="36.195" x2="35.56" y2="36.83" width="0.4064" layer="16"/>
+<wire x1="35.56" y1="36.83" x2="35.56" y2="40.005" width="0.4064" layer="16"/>
+<wire x1="35.56" y1="40.005" x2="34.395" y2="41.17" width="0.4064" layer="16"/>
+<wire x1="34.395" y1="41.17" x2="33.74" y2="41.17" width="0.4064" layer="16"/>
+<wire x1="35.56" y1="40.005" x2="39.8779" y2="41.4516" width="0" layer="19" extent="1-16"/>
 </signal>
 <signal name="N$32">
 <contactref element="C10" pad="2"/>
 <contactref element="U$1" pad="20"/>
-<wire x1="43.815" y1="33.67" x2="41.4196" y2="41.4516" width="0" layer="19" extent="1-1"/>
+<wire x1="43.815" y1="33.67" x2="43.815" y2="36.195" width="0.4064" layer="1"/>
+<wire x1="43.815" y1="36.195" x2="43.18" y2="36.83" width="0.4064" layer="1"/>
+<via x="43.18" y="36.83" extent="1-16" drill="0.6"/>
+<wire x1="43.18" y1="36.83" x2="43.18" y2="41.91" width="0.4064" layer="16"/>
+<wire x1="43.18" y1="41.91" x2="41.91" y2="43.18" width="0.4064" layer="16"/>
+<via x="41.91" y="43.18" extent="1-16" drill="0.6"/>
+<wire x1="41.91" y1="43.18" x2="41.4196" y2="42.6896" width="0.4064" layer="1"/>
+<wire x1="41.4196" y1="42.6896" x2="41.4196" y2="41.4516" width="0.4064" layer="1"/>
 </signal>
 <signal name="N$29">
@@
 <contactref element="U$3" pad="ADC"/>
 <contactref element="S1" pad="1"/>
-<wire x1="9.525" y1="68.58" x2="19.685" y2="58.42" width="1.27" layer="16"/>
-<wire x1="19.685" y1="58.42" x2="25.4" y2="58.42" width="1.27" layer="16"/>
-<wire x1="25.4" y1="58.42" x2="32.385" y2="51.435" width="1.27" layer="16"/>
-<wire x1="32.385" y1="51.435" x2="36.83" y2="46.99" width="1.27" layer="16"/>
-<wire x1="36.83" y1="46.99" x2="36.83" y2="31.75" width="1.27" layer="16"/>
-<wire x1="36.83" y1="31.75" x2="39.37" y2="29.21" width="1.27" layer="16"/>
+<wire x1="9.525" y1="68.58" x2="13.97" y2="64.77" width="1.27" layer="16"/>
+<wire x1="13.97" y1="64.77" x2="19.05" y2="64.77" width="1.27" layer="16"/>
+<wire x1="19.05" y1="64.77" x2="32.385" y2="51.435" width="1.27" layer="16"/>
+<wire x1="32.385" y1="51.435" x2="37.465" y2="46.355" width="1.27" layer="16"/>
+<wire x1="37.465" y1="46.355" x2="37.465" y2="31.115" width="1.27" layer="16"/>
+<wire x1="37.465" y1="31.115" x2="39.37" y2="29.21" width="1.27" layer="16"/>
 <wire x1="39.37" y1="29.21" x2="39.37" y2="27.94" width="1.27" layer="16"/>
 <wire x1="70.485" y1="68.58" x2="53.34" y2="51.435" width="1.27" layer="16"/>
-<wire x1="53.34" y1="51.435" x2="53.34" y2="26.67" width="1.27" layer="16"/>
+<wire x1="53.34" y1="51.435" x2="53.34" y2="43.18" width="1.27" layer="16"/>
+<wire x1="53.34" y1="43.18" x2="53.34" y2="26.67" width="1.27" layer="16"/>
 <wire x1="53.34" y1="26.67" x2="52.705" y2="26.035" width="1.27" layer="16"/>
 <wire x1="52.705" y1="26.035" x2="41.275" y2="26.035" width="1.27" layer="16"/>
 <wire x1="41.275" y1="26.035" x2="39.37" y2="27.94" width="1.27" layer="16"/>
-<wire x1="70.485" y1="11.43" x2="55.88" y2="26.035" width="1.27" layer="16"/>
-<wire x1="55.88" y1="26.035" x2="52.705" y2="26.035" width="1.27" layer="16"/>
+<wire x1="70.485" y1="11.43" x2="67.31" y2="13.97" width="1.27" layer="16"/>
+<wire x1="67.31" y1="13.97" x2="63.5" y2="13.97" width="1.27" layer="16"/>
+<wire x1="63.5" y1="13.97" x2="52.705" y2="24.765" width="1.27" layer="16"/>
+<wire x1="52.705" y1="24.765" x2="52.705" y2="26.035" width="1.27" layer="16"/>
 <wire x1="31.43" y1="48.9251" x2="31.43" y2="49.845" width="0.6096" layer="1"/>
 <wire x1="31.43" y1="49.845" x2="31.75" y2="50.165" width="0.6096" layer="1"/>
@@
 <via x="26.67" y="26.67" extent="1-16" drill="0.6" shape="octagon"/>
 <wire x1="26.67" y1="26.67" x2="26.67" y2="26.035" width="1.27" layer="16"/>
-<wire x1="53.34" y1="51.435" x2="47.74" y2="43.17" width="0" layer="19" extent="16-16"/>
+<wire x1="47.74" y1="43.17" x2="47.75" y2="43.18" width="0.4064" layer="16"/>
+<wire x1="47.75" y1="43.18" x2="53.34" y2="43.18" width="0.4064" layer="16"/>
 </signal>
 <signal name="SDA">
@@
 <wire x1="39.3733" y1="41.4516" x2="38.9149" y2="41.91" width="0.4064" layer="1"/>
 <wire x1="38.9149" y1="41.91" x2="38.1" y2="41.91" width="0.4064" layer="1"/>
-<wire x1="38.1" y1="41.91" x2="36.195" y2="40.005" width="0.4064" layer="1"/>
-<wire x1="36.195" y1="40.005" x2="35.36" y2="39.17" width="0.4064" layer="1"/>
-<wire x1="35.36" y1="39.17" x2="33.74" y2="39.17" width="0.4064" layer="1"/>
-<wire x1="36.195" y1="33.67" x2="36.195" y2="40.005" width="0.4064" layer="1"/>
+<wire x1="38.1" y1="41.91" x2="35.36" y2="39.17" width="0.4064" layer="1"/>
+<wire x1="35.36" y1="39.17" x2="34.925" y2="39.17" width="0.4064" layer="1"/>
+<wire x1="34.925" y1="39.17" x2="33.74" y2="39.17" width="0.4064" layer="1"/>
+<wire x1="36.195" y1="33.67" x2="34.94" y2="34.925" width="0.4064" layer="1"/>
+<wire x1="34.94" y1="34.925" x2="34.925" y2="34.925" width="0.4064" layer="1"/>
+<wire x1="34.925" y1="34.925" x2="34.925" y2="39.17" width="0.4064" layer="1"/>
 </signal>
 <signal name="N$38">
@@
 <contactref element="U$3" pad="GPIO16"/>
 <wire x1="61.135378125" y1="62.405378125" x2="62.405378125" y2="61.135378125" width="0.4064" layer="1"/>
-<wire x1="47.74" y1="39.17" x2="53.14" y2="39.17" width="0.4064" layer="1"/>
-<wire x1="53.14" y1="39.17" x2="54.61" y2="40.64" width="0.4064" layer="1"/>
-<wire x1="54.61" y1="40.64" x2="54.61" y2="53.34" width="0.4064" layer="1"/>
-<wire x1="54.61" y1="53.34" x2="62.405378125" y2="61.135378125" width="0.4064" layer="1"/>
+<wire x1="47.74" y1="39.17" x2="51.235" y2="39.17" width="0.4064" layer="1"/>
+<wire x1="51.235" y1="39.17" x2="51.435" y2="39.37" width="0.4064" layer="1"/>
+<wire x1="51.435" y1="39.37" x2="51.435" y2="50.165" width="0.4064" layer="1"/>
+<wire x1="51.435" y1="50.165" x2="62.405378125" y2="61.135378125" width="0.4064" layer="1"/>
 </signal>
 <signal name="M3">
@@
 <wire x1="42.7262" y1="38.0733" x2="44.6433" y2="38.0733" width="0.4064" layer="1"/>
 <wire x1="44.6433" y1="38.0733" x2="47.74" y2="41.17" width="0.4064" layer="1"/>
+<wire x1="47.74" y1="31.17" x2="51.49" y2="31.17" width="0.4064" layer="16"/>
+<wire x1="51.49" y1="31.17" x2="52.07" y2="31.75" width="0.4064" layer="16"/>
+<wire x1="52.07" y1="31.75" x2="52.07" y2="39.37" width="0.4064" layer="16"/>
+<wire x1="52.07" y1="39.37" x2="50.27" y2="41.17" width="0.4064" layer="16"/>
+<wire x1="50.27" y1="41.17" x2="47.74" y2="41.17" width="0.4064" layer="16"/>
 <wire x1="31.13" y1="52.07" x2="31.43" y2="46.3249" width="0" layer="19" extent="1-1"/>
 <wire x1="33.74" y1="35.17" x2="31.43" y2="46.3249" width="0" layer="19" extent="1-1"/>
 <wire x1="42.7262" y1="38.0733" x2="38.735" y2="32.37" width="0" layer="19" extent="1-1"/>
-<wire x1="47.74" y1="31.17" x2="44.6433" y2="38.0733" width="0" layer="19" extent="1-1"/>
 </signal>
 <signal name="N$1">

Commit message: pcb update
Parts:
- moved R1 5.85 mm to (34.9, 31.8), turned to 90 degrees
- moved C14 2.29 mm to (44.5, 31.8)
- moved C10 1.80 mm to (42.5, 31.8)
- moved C6 1.42 mm to (40.6, 31.8)
- moved R5 1.42 mm to (36.8, 31.8)
- moved R4 1.27 mm to (38.7, 31.8)
- turned C2 to 0 degrees
- turned R10 to 225 degrees
- turned R12 to 315 degrees
- turned R14 to 45 degrees
Routing:
- net GND: track 174.2 -> 248.7 mm, vias 0 -> 2
- net M2: track 1.80 -> 63.7 mm
- net M1: track 1.80 -> 52.2 mm, vias 0 -> 1
- net 3.3V: track 37.7 -> 74.6 mm, vias 0 -> 3
- net TX: track 0.00 -> 29.9 mm, vias 0 -> 1
- net RX: track 0.00 -> 29.1 mm, vias 0 -> 1
- net M3: track 1.80 -> 26.5 mm, vias 0 -> 2
- net DTR: track 22.5 -> 35.5 mm, vias 2 -> 1
- net SCL: track 9.96 -> 19.4 mm, vias 1 -> 2
- net N$20: track 7.40 -> 1.50 mm
- net N$5: track 9.61 -> 14.5 mm
- net VCC: track 207.1 -> 209.6 mm, vias 3 -> 4
- net SDA: track 13.0 -> 15.4 mm, vias 0 -> 2
- net N$29: track 3.73 -> 4.96 mm
- net M4: track 31.9 -> 33.0 mm, vias 0 -> 2
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