File: hardware/Flying5 v1.0 - schematic design/Flying5.brd (EAGLE design)
At the start: 83.2 x 83.2 mm, 30 parts, among them Q1 IRLML2502, Q2 IRLML2502, Q3 IRLML2502, Q4 IRLML2502, U2 MIC5205

Commit message: update sch
Parts:
- removed S1: (no value), SparkFun-Electromechanical:SWITCH-SPDT-SMD
- removed U$3: ESP12, esp8266modules:ESP12
- added ESP12E: (no value), esp8266modules:ESP12E-SMD
- added J1: 短路点, SparkFun-Connectors:1X02
- added U$2: SWITCH_SK12D07, example:SK12D07
- moved POWER 31.8 mm to (55.2, 54.0), turned to 135 degrees
- moved FTDI 17.3 mm to (26.7, 38.1), turned to 270 degrees
- moved C1 8.52 mm to (22.9, 57.1), turned to 135 degrees
- moved C2 4.02 mm to (26.7, 53.3), turned to 225 degrees
- moved R1 3.59 mm to (37.5, 29.2), turned to 45 degrees
- moved U2 3.42 mm to (29.2, 50.8), turned to 225 degrees
- moved R4 2.84 mm to (41.3, 33.0), turned to 225 degrees
- moved C10 2.84 mm to (43.8, 29.2), turned to 45 degrees
- moved C6 2.54 mm to (40.6, 29.2), turned to 45 degrees
- moved R5 1.80 mm to (38.1, 33.0), turned to 45 degrees
- moved C14 1.27 mm to (44.5, 33.0), turned to 225 degrees
Connections:
- removed net N$20: R1.2, U$3.GPIO15
- new net CTS: FTDI.P$5
- new net GPIO0: ESP12E.GPIO0, J1.2
- net 3.3V: now also ESP12E.CH_PD, ESP12E.VCC; no longer U$3.CH_PD, U$3.GPIO2, U$3.VCC
- net DTR: now also ESP12E.RESET; no longer U$3.GPIO0
- net GND: now also ESP12E.GND, J1.1; no longer FTDI.P$5, U$3.GND
- net M1: now also ESP12E.GPIO14; no longer U$3.GPIO14
- net M2: now also ESP12E.GPIO12; no longer U$3.GPIO12
- net M3: now also ESP12E.GPIO13; no longer U$3.GPIO13
- net M4: now also ESP12E.GPIO15, R1.2; no longer U$3.GPIO16
- net N$6: now also U$2.2; no longer S1.2
- net RX: now also ESP12E.RXD0, FTDI.P$3; no longer FTDI.P$2, U$3.RX
- net SCL: now also ESP12E.GPIO5; no longer U$3.GPIO4
- net SDA: now also ESP12E.GPIO4; no longer U$3.GPIO5
- net TX: now also ESP12E.TXD0, FTDI.P$2; no longer FTDI.P$3, U$3.TX
- net VCC: now also ESP12E.ADC, U$2.1; no longer S1.1, U$3.ADC
Routing:
- net TX: track 29.9 -> 2.61 mm, vias 1 -> 0
- net GND: track 248.7 -> 226.4 mm, vias 2 -> 5
- net RX: track 29.1 -> 10.8 mm, vias 1 -> 0
- net DTR: track 35.5 -> 19.8 mm, vias 1 -> 0
- net VCC: track 209.6 -> 222.5 mm, vias 4 -> 1
- net SCL: track 19.4 -> 27.9 mm, vias 2 -> 1
- net 3.3V: track 74.6 -> 82.6 mm, vias 3 -> 6
- net N$32: track 13.1 -> 19.3 mm, vias 2 -> 0
- net M4: track 33.0 -> 38.6 mm, vias 2 -> 4
- net M2: track 63.7 -> 68.9 mm, vias 0 -> 1
- net M3: track 26.5 -> 21.3 mm, vias 2 -> 1
- net N$5: track 14.5 -> 9.40 mm, vias 2 -> 0
- net N$29: track 4.96 -> 9.47 mm, vias 0 -> 2
- net SDA: track 15.4 -> 19.3 mm, vias 2 -> 1
- net M1: track 52.2 -> 55.6 mm
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- added copper zone on layer 16, net N$10
- added copper zone on layer 1, net N$9
Other:
- board text added: "www.flying5.com"
- board text removed: "+"
- board text removed: "Flying5"

Commit message: update pcb
Parts:
- added R2: 1K, SparkFun-Passives:0402-RES
Connections:
- new net N$15: R2.2, U$1.9
- net GND: now also R2.1
Changed lines of the file:
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@@
 <element name="U$2" library="example" package="SK12D07" value="SWITCH_SK12D07" x="40.64" y="53.34"/>
 <element name="J1" library="SparkFun-Connectors" package="1X02" value="短路点" x="-11.43" y="0"/>
+<element name="R2" library="SparkFun-Passives" package="0402-RES" value="1K" x="-11.43" y="-6.35"/>
 </elements>
 <signals>
@@
 <wire x1="44.90961875" y1="33.655" x2="44.90961875" y2="33.47961875" width="0.3048" layer="1"/>
 <contactref element="J1" pad="1"/>
+<contactref element="R2" pad="1"/>
 <wire x1="-11.43" y1="0" x2="14.076065625" y2="15.41956875" width="0" layer="19" extent="1-1"/>
+<wire x1="-12.08" y1="-6.35" x2="-11.43" y2="0" width="0" layer="19" extent="1-1"/>
 </signal>
 <signal name="DTR">
@@
 <wire x1="-8.89" y1="0" x2="32.54" y2="34.63" width="0" layer="19" extent="16-16"/>
 </signal>
+<signal name="N$15">
+<contactref element="U$1" pad="9"/>
+<contactref element="R2" pad="2"/>
+<wire x1="-10.78" y1="-6.35" x2="40.3825" y2="37.2484" width="0" layer="19" extent="1-1"/>
+</signal>
 </signals>

Commit message: pcb update
Parts:
- removed R2: 1K, SparkFun-Passives:0402-RES
- removed U$2: SWITCH_SK12D07, example:SK12D07
- added S1: (no value), SparkFun-Electromechanical:SWITCH-SPST-SMD-A
- J1: value 短路点 -> 短接点
- moved J1 44.5 mm to (24.1, 26.7)
- turned C10 to 225 degrees
- turned R4 to 45 degrees
- renumbered Q1 to MOTOR4, Q2 to MOTOR3, Q3 to MOTOR2, Q4 to MOTOR1
Connections:
- removed net N$15: R2.2, U$1.9
- new net N$16: ESP12E.GPIO15, R1.2
- net GND: no longer R2.1
- net M1: now also ESP12E.GPIO5; no longer ESP12E.GPIO14
- net M2: now also ESP12E.GPIO4; no longer ESP12E.GPIO12
- net M4: now also ESP12E.GPIO14; no longer ESP12E.GPIO15, R1.2
- net N$6: now also S1.2; no longer U$2.2
- net SCL: now also ESP12E.GPIO12; no longer ESP12E.GPIO5
- net SDA: now also ESP12E.GPIO2; no longer ESP12E.GPIO4
- net VCC: now also S1.1; no longer U$2.1
Routing:
- net GND: track 226.4 -> 0.00 mm, vias 5 -> 0
- net VCC: track 222.5 -> 0.00 mm, vias 1 -> 0
- net 3.3V: track 82.6 -> 0.00 mm, vias 6 -> 0
- net M2: track 68.9 -> 0.00 mm, vias 1 -> 0
- net M1: track 55.6 -> 0.00 mm, vias 1 -> 0
- net M4: track 38.6 -> 0.00 mm, vias 4 -> 0
- net SCL: track 27.9 -> 0.00 mm, vias 1 -> 0
- net M3: track 21.3 -> 0.00 mm, vias 1 -> 0
- net DTR: track 19.8 -> 0.00 mm
- net SDA: track 19.3 -> 0.00 mm, vias 1 -> 0
- net N$32: track 19.3 -> 0.00 mm
- net N$6: track 16.7 -> 0.00 mm
- net RX: track 10.8 -> 0.00 mm
- net N$29: track 9.47 -> 0.00 mm, vias 2 -> 0
- net N$5: track 9.40 -> 0.00 mm
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
Commit message: gen gerber
Parts:
- moved J1 2.84 mm to (26.7, 25.4)
- moved POWER 1.80 mm to (54.0, 52.7)
- moved R7 0.63 mm to (16.5, 62.2)
- moved R8 0.63 mm to (17.8, 63.5)
- turned R10 to 45 degrees
- turned R12 to 135 degrees
- turned R14 to 225 degrees
Routing:
- net GND: track 0.00 -> 238.0 mm, vias 0 -> 2
- net VCC: track 0.00 -> 210.0 mm, vias 0 -> 3
- net 3.3V: track 0.00 -> 76.5 mm, vias 0 -> 3
- net M1: track 0.00 -> 37.8 mm, vias 0 -> 1
- net M4: track 0.00 -> 35.9 mm, vias 0 -> 1
- net M2: track 0.00 -> 27.6 mm, vias 0 -> 1
- net DTR: track 0.00 -> 24.1 mm, vias 0 -> 2
- net N$32: track 0.00 -> 23.6 mm, vias 0 -> 2
- net SCL: track 0.00 -> 21.8 mm, vias 0 -> 2
- net M3: track 0.00 -> 20.9 mm, vias 0 -> 1
- net SDA: track 0.00 -> 18.2 mm, vias 0 -> 2
- net N$6: track 0.00 -> 17.1 mm
- net N$5: track 0.00 -> 12.2 mm, vias 0 -> 2
- net GPIO0: track 0.00 -> 12.0 mm
- net N$29: track 0.00 -> 9.38 mm
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