File: hardware/Flying5 v1.0 - schematic design/Flying5.sch (EAGLE design)
At the start: 30 parts, among them Q1 IRLML2502, Q2 IRLML2502, Q3 IRLML2502, Q4 IRLML2502, U2 MIC5205

Commit message: update sch
Parts:
- removed S1: (no value), SparkFun-Electromechanical:SWITCH-SPDTSMD2
- removed U$3: ESP12, esp8266modules:ESP12
- added ESP12E: (no value), esp8266modules:ESP12ESMD
- added J1: 短路点, SparkFun-Connectors:M02PTH
- added U$2: SWITCH_SK12D07, example:SWITCH_SK12D07
- POWER: value M02PTH -> (none)
Connections:
- removed net N$20: R1.2, U$3.GPIO15
- new net CTS: FTDI.CTS
- new net GPIO0: ESP12E.GPIO0, J1.2
- net 3.3V: now also ESP12E.CH_PD, ESP12E.VCC; no longer U$3.CH_PD, U$3.GPIO2, U$3.VCC
- net DTR: now also ESP12E.RESET; no longer U$3.GPIO0
- net GND: now also ESP12E.GND, J1.1; no longer FTDI.CTS, U$3.GND
- net M1: now also ESP12E.GPIO14; no longer U$3.GPIO14
- net M2: now also ESP12E.GPIO12; no longer U$3.GPIO12
- net M3: now also ESP12E.GPIO13; no longer U$3.GPIO13
- net M4: now also ESP12E.GPIO15, R1.2; no longer U$3.GPIO16
- net N$6: now also U$2.P; no longer S1.P
- net RX: now also ESP12E.RX, FTDI.RXI; no longer FTDI.TXO, U$3.RX
- net SCL: now also ESP12E.GPIO5; no longer U$3.GPIO4
- net SDA: now also ESP12E.GPIO4; no longer U$3.GPIO5
- net TX: now also ESP12E.TX, FTDI.TXO; no longer FTDI.RXI, U$3.TX
- net VCC: now also ESP12E.ADC, U$2.O; no longer S1.O, U$3.ADC
Other:
- moved on the sheet: R1

Commit message: update pcb
Parts:
- added R2: 1K, SparkFun-Passives:RESISTOR0402-RES
Connections:
- new net N$15: R2.2, U$1.AD0
- net GND: now also R2.1
Changed lines of the file:
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@@
 <part name="J1" library="SparkFun-Connectors" deviceset="M02" device="PTH" value="短路点"/>
 <part name="GND7" library="SparkFun-Aesthetics" deviceset="GND" device=""/>
+<part name="R2" library="SparkFun-Passives" deviceset="RESISTOR" device="0402-RES" value="1K"/>
+<part name="GND12" library="SparkFun-Aesthetics" deviceset="GND" device=""/>
 </parts>
 <sheets>
@@
 <instance part="J1" gate="G$1" x="-50.8" y="76.2"/>
 <instance part="GND7" gate="1" x="-38.1" y="68.58"/>
+<instance part="R2" gate="G$1" x="12.7" y="-68.58" rot="R90"/>
+<instance part="GND12" gate="1" x="12.7" y="-78.74"/>
 </instances>
 <busses>
@@
 <wire x1="-38.1" y1="76.2" x2="-38.1" y2="71.12" width="0.1524" layer="91"/>
 <pinref part="GND7" gate="1" pin="GND"/>
+</segment>
+<segment>
+<pinref part="R2" gate="G$1" pin="1"/>
+<pinref part="GND12" gate="1" pin="GND"/>
+<wire x1="12.7" y1="-73.66" x2="12.7" y2="-76.2" width="0.1524" layer="91"/>
 </segment>
 </net>
@@
 </segment>
 </net>
+<net name="N$15" class="0">
+<segment>
+<pinref part="U$1" gate="G$1" pin="AD0"/>
+<wire x1="-10.16" y1="-60.96" x2="12.7" y2="-60.96" width="0.1524" layer="91"/>
+<wire x1="12.7" y1="-60.96" x2="12.7" y2="-63.5" width="0.1524" layer="91"/>
+<pinref part="R2" gate="G$1" pin="2"/>
+</segment>
+</net>

Commit message: pcb update
Parts:
- removed R2: 1K, SparkFun-Passives:RESISTOR0402-RES
- removed U$2: SWITCH_SK12D07, example:SWITCH_SK12D07
- added S1: (no value), SparkFun-Electromechanical:SWITCH-SPDT-SMD-A
- J1: value 短路点 -> 短接点
- renumbered Q1 to MOTOR4, Q2 to MOTOR3, Q3 to MOTOR2, Q4 to MOTOR1
Connections:
- removed net N$15: R2.2, U$1.AD0
- new net N$16: ESP12E.GPIO15, R1.2
- net GND: no longer R2.1
- net M1: now also ESP12E.GPIO5; no longer ESP12E.GPIO14
- net M2: now also ESP12E.GPIO4; no longer ESP12E.GPIO12
- net M4: now also ESP12E.GPIO14; no longer ESP12E.GPIO15, R1.2
- net N$6: now also S1.P; no longer U$2.P
- net SCL: now also ESP12E.GPIO12; no longer ESP12E.GPIO5
- net SDA: now also ESP12E.GPIO2; no longer ESP12E.GPIO4
- net VCC: now also S1.O; no longer U$2.O
